Commit message: Ajout des subscribers

File: desherbor_ensta/urdf/robot.lidar.xacro (robot description, xacro)
@@ -5,5 +5,5 @@
     <sensor type="ray" name="lidar_sensor">
       <pose>0 0 0 0 0 0</pose>
-      <visualize>false</visualize>
+      <visualize>true</visualize>
       <update_rate>5</update_rate>
       <ray>

File: desherbor_ensta/urdf/robot_desherbor.urdf.xacro (robot description, xacro)
@@ -166,5 +166,5 @@
   <link name="lidar">
     <visual>
-      <origin xyz="0 0 0.075" rpy="0 0 0"/>
+      <origin xyz="0 0 -0.03" rpy="0 0 0"/>
       <geometry>
         <cylinder radius="0.03" length="0.1"/>
@@ -175,6 +175,6 @@
   <joint name="lidar_hinge" type="fixed">
     <child link="lidar"/>
-    <parent link="arm"/>
-    <origin xyz="0 0 0.075" rpy="0 0 0"/>
+    <parent link="chassis"/>
+    <origin xyz="0 0 0.22" rpy="0 0 0"/>
   </joint>
     <link name="camera">
@@ -248,5 +248,5 @@
   <link name="imu_link">
     <visual>
-      <origin xyz="0 0 0.1" rpy="0 0 0"/>
+      <origin xyz="0 0 0.01" rpy="0 0 0"/>
       <geometry>
         <cylinder radius="0.01" length="0.01"/>
