Commit message: robot OK bras OK

File: desherbor_ensta/urdf/robot_desherbor.urdf.xacro (robot description, xacro)
@@ -24,8 +24,8 @@
       <origin xyz="0 0 .1" rpy="0 0 0"/>
       <geometry>
-        <box size="0.3 0.3 0.1"/>
+        <box size="0.1 0.3 0.1"/>
       </geometry>
     </visual>
-    <xacro:default_inertial mass="2.0"/>
+    <xacro:default_inertial mass="4.0"/>
   </link>
   <link name="left_top_wheel">
@@ -115,22 +115,22 @@
   <link name="arm">
     <collision>
-      <origin xyz="0 0 0" rpy="0 1.5707 1.5707"/>
+      <origin xyz="0.2 0 0.2" rpy="0 1.56 0"/>
       <geometry>
-        <cylinder radius="0.05" length="0.3"/>
+        <cylinder radius="0.01" length="0.3"/>
       </geometry>
     </collision>
     <visual>
-      <origin xyz="0 0 0" rpy="0 1.5707 1.5707"/>
+      <origin xyz="0.2 0 0.2" rpy="0 1.56 0"/>
       <geometry>
-        <cylinder radius="0.1" length="0.05"/>
+        <cylinder radius="0.01" length="0.3"/>
       </geometry>
     </visual>
-    <xacro:default_inertial mass="0.2"/>
+    <xacro:default_inertial mass="0.1"/>
   </link>
   <joint type="continuous" name="arm_hinge">
-    <origin xyz="1.15 1.15 0.1" rpy="0 0 0"/>
+    <origin xyz="0 0 0" rpy="0 0 0"/>
     <child link="arm"/>
     <parent link="chassis"/>
-    <axis xyz="0 1 0"/>
+    <axis xyz="0 0 1"/>
   </joint>
 </robot>

Commit message: Ajout des controllers

File: desherbor_ensta/urdf/robot_desherbor.urdf.xacro (robot description, xacro)
@@ -93,5 +93,5 @@
     <child link="left_top_wheel"/>
     <parent link="chassis"/>
-    <axis xyz="0 1 0"/>
+    <axis xyz="0 0 1"/>
   </joint>
   <joint type="continuous" name="right_top_wheel_hinge">
@@ -99,5 +99,5 @@
     <child link="right_top_wheel"/>
     <parent link="chassis"/>
-    <axis xyz="0 1 0"/>
+    <axis xyz="0 0 1"/>
   </joint>
   <joint type="continuous" name="left_bottom_wheel_hinge">
@@ -182,3 +182,48 @@
     <origin xyz="0.2 0 0.1" rpy="0 0 0"/>
   </joint>
+  <transmission name="trans_left_bottom_wheel">
+    <type> transmission_interface/SimpleTransmission </type>
+    <joint name="left_bottom_wheel_hinge">
+      <hardwareInterface> EffortJointInterface</hardwareInterface>
+    </joint>
+    <actuator name="bottom_wheel_actuator">
+      <mechanicalReduction>50</mechanicalReduction>
+      <hardwareInterface>EffortJointInterface</hardwareInterface>
+    </actuator>
+  </transmission>
+  <transmission name="trans_right_bottom_wheel">
+    <type> transmission_interface/SimpleTransmission </type>
+    <joint name="right_bottom_wheel_hinge">
+      <hardwareInterface>EffortJointInterface</hardwareInterface>
+    </joint>
+    <actuator name="bottom_wheel_actuator">
+      <mechanicalReduction>50</mechanicalReduction>
+      <hardwareInterface>EffortJointInterface</hardwareInterface>
+    </actuator>
+  </transmission>
+  <transmission name="trans_left_top_wheel">
+    <type> transmission_interface/SimpleTransmission</type>
+    <joint name="left_top_wheel_hinge">
+      <hardwareInterface>EffortJointInterface</hardwareInterface>
+    </joint>
+    <actuator name="top_wheel_actuator">
+      <mechanicalReduction>30</mechanicalReduction>
+      <hardwareInterface>EffortJointInterface</hardwareInterface>
+    </actuator>
+  </transmission>
+  <transmission name="trans_right_top_wheel">
+    <type> transmission_interface/SimpleTransmission</type>
+    <joint name="right_top_wheel_hinge">
+      <hardwareInterface>EffortJointInterface</hardwareInterface>
+    </joint>
+    <actuator name="top_wheel_actuator">
+      <mechanicalReduction>30</mechanicalReduction>
+      <hardwareInterface>EffortJointInterface</hardwareInterface>
+    </actuator>
+  </transmission>
+  <gazebo>
+    <plugin name="gazebo_ros_control" filename="libgazebo_ros_control.so">
+      <robotNamespace>/desherbor_ensta</robotNamespace>
+    </plugin>
+  </gazebo>
 </robot>

Commit message: Ajout controleur pour le bras

File: desherbor_ensta/urdf/robot_desherbor.urdf.xacro (robot description, xacro)
@@ -222,4 +222,14 @@
     </actuator>
   </transmission>
+  <transmission name="trans_arm">
+    <type> transmission_interface/SimpleTransmission</type>
+    <joint name="arm_hinge">
+      <hardwareInterface>EffortJointInterface</hardwareInterface>
+    </joint>
+    <actuator name="arm_actuator">
+      <mechanicalReduction>30</mechanicalReduction>
+      <hardwareInterface>EffortJointInterface</hardwareInterface>
+    </actuator>
+  </transmission>
   <gazebo>
     <plugin name="gazebo_ros_control" filename="libgazebo_ros_control.so">

Commit message: modilisation de la camera

File: desherbor_ensta/urdf/robot_desherbor.urdf.xacro (robot description, xacro)
@@ -2,4 +2,5 @@
 <robot name = "desherbor_ensta" xmlns:xacro="http://ros.org/wiki/xacro">
   <xacro:include filename="$(find desherbor_ensta)/urdf/robot_desherbor.wheels.xacro"/>
+  <xacro:include filename="$(find desherbor_ensta)/urdf/robot_desherbor.camera.xacro"/>
   <xacro:macro name="default_inertial" params="mass">
     <inertial>
@@ -89,4 +90,12 @@
     <xacro:default_inertial mass="0.3"/>
   </link>
+  <link name="camera">
+    <visual>
+      <geometry>
+        <sphere radius="0.01"/>
+      </geometry>
+    </visual>
+    <xacro:default_inertial mass="0.01"/>
+  </link>
   <joint type="continuous" name="left_top_wheel_hinge">
     <origin xyz="0.1 0.13 0.1" rpy="0 0 0"/>
@@ -133,4 +142,9 @@
     <parent link="chassis"/>
     <axis xyz="0 0 1"/>
+  </joint>
+  <joint name="camera_joint" type="fixed">
+    <parent link="chassis"/>
+    <child link="camera"/>
+    <origin xyz="0.1 0.0 0.1" rpy="0 0 0"/>
   </joint>
   <link name="laser">

Commit message: placement du robot et du lidar

File: desherbor_ensta/urdf/robot_desherbor.urdf.xacro (robot description, xacro)
@@ -136,13 +136,13 @@
   <link name="laser">
     <collision>
-      <origin xyz="0 0 0" rpy="0 1.5707 1.5707"/>
+      <origin xyz="0.16 0 0.095" rpy="0 0 1.5707"/>
       <geometry>
-        <cylinder radius="0.025" length="0.15"/>
+        <cylinder radius="0.025" length="0.017"/>
       </geometry>
     </collision>
     <visual>
-      <origin xyz="0 0 0" rpy="0 1.5707 1.5707"/>
+      <origin xyz="0.16 0 0.095" rpy="0 0 1.5707"/>
       <geometry>
-        <cylinder radius="0.05" length="0.15"/>
+        <cylinder radius="0.0025" length="0.017"/>
       </geometry>
     </visual>
@@ -150,5 +150,5 @@
   </link>
   <joint type="fixed" name="laser_hinge">
-    <origin xyz="-0.1 -0.13 0.1" rpy="0 0 0"/>
+    <origin xyz="0.16 0 0.095" rpy="0 0 0"/>
     <child link="laser"/>
     <parent link="arm"/>
@@ -157,5 +157,5 @@
   <link name="lidar">
     <visual>
-      <origin xyz="0 0 -0.03" rpy="0 0 0"/>
+      <origin xyz="0 0 0.075" rpy="0 0 0"/>
       <geometry>
         <cylinder radius="0.03" length="0.1"/>
@@ -167,18 +167,5 @@
     <child link="lidar"/>
     <parent link="arm"/>
-    <origin xyz="0.15 0 0.23" rpy="0 0 0"/>
-  </joint>
-  <link name="camera">
-    <visual>
-      <geometry>
-        <sphere radius="0.01"/>
-      </geometry>
-    </visual>
-    <xacro:default_inertial mass="0.01"/>
-  </link>
-  <joint name="camera_hinge" type="fixed">
-    <child link="camera"/>
-    <parent link="arm"/>
-    <origin xyz="0.2 0 0.1" rpy="0 0 0"/>
+    <origin xyz="0 0 0.075" rpy="0 0 0"/>
   </joint>
 </robot>

Commit message: minor change

File: desherbor_ensta/urdf/robot_desherbor.urdf.xacro (robot description, xacro)
@@ -18,11 +18,11 @@
       <origin xyz="0 0 .1" rpy="0 0 0"/>
       <geometry>
+        <box size="0.1 0.3 0.1"/>
+      </geometry>
+    </collision>
+    <visual>
+      <origin xyz="0 0 .1" rpy="0 0 0"/>
+      <geometry>
         <box size="0.3 0.3 0.1"/>
-      </geometry>
-    </collision>
-    <visual>
-      <origin xyz="0 0 .1" rpy="0 0 0"/>
-      <geometry>
-        <box size="0.1 0.3 0.1"/>
       </geometry>
     </visual>

Commit message: Positionnement de l'IMU au milieu du robot

File: desherbor_ensta/urdf/robot_desherbor.urdf.xacro (robot description, xacro)
@@ -93,12 +93,4 @@
     <xacro:default_inertial mass="0.3"/>
   </link>
-  <link name="camera">
-    <visual>
-      <geometry>
-        <sphere radius="0.01"/>
-      </geometry>
-    </visual>
-    <xacro:default_inertial mass="0.01"/>
-  </link>
   <joint type="continuous" name="left_top_wheel_hinge">
     <origin xyz="0.1 0.13 0.1" rpy="0 0 0"/>
@@ -256,8 +248,13 @@
   <link name="imu_link">
     <visual>
-      <origin xyz="0 0 -0.03" rpy="0 0 0"/>
-      <geometry>
-        <cylinder radius="0.03" length="0.1"/>
-      </geometry>
+      <origin xyz="0 0 0.1" rpy="0 0 0"/>
+      <geometry>
+        <cylinder radius="0.01" length="0.01"/>
+      </geometry>
+      <collision>
+        <geometry>
+          <cylinder radius="0.001" length="0.001"/>
+        </geometry>
+      </collision>
     </visual>
     <xacro:default_inertial mass="0.1"/>
@@ -266,5 +263,5 @@
     <child link="imu_link"/>
     <parent link="chassis"/>
-    <origin xyz="0 0 -0.03" rpy="0 0 0"/>
+    <origin xyz="0 0 0.1" rpy="0 0 0"/>
   </joint>
 </robot>

Commit message: Ajout de la caméra

File: desherbor_ensta/urdf/robot_desherbor.urdf.xacro (robot description, xacro)
@@ -178,4 +178,12 @@
     <origin xyz="0 0 0.075" rpy="0 0 0"/>
   </joint>
+    <link name="camera">
+    <visual>
+      <geometry>
+        <sphere radius="0.01"/>
+      </geometry>
+    </visual>
+    <xacro:default_inertial mass="0.01"/>
+  </link>
   <joint name="camera_hinge" type="fixed">
     <child link="camera"/>

Commit message: ajout position laser

File: desherbor_ensta/urdf/robot_desherbor.urdf.xacro (robot description, xacro)
@@ -183,14 +183,4 @@
     <origin xyz="0 0 0.075" rpy="0 0 0"/>
   </joint>
-<<<<<<< HEAD
-=======
-  <link name="camera">
-    <visual>
-      <geometry>
-        <sphere radius="0.01"/>
-      </geometry>
-    </visual>
-    <xacro:default_inertial mass="0.01"/>
-  </link>
   <joint name="camera_hinge" type="fixed">
     <child link="camera"/>
@@ -253,4 +243,3 @@
     </plugin>
   </gazebo>
->>>>>>> master
 </robot>

Commit message: change collision size

File: desherbor_ensta/urdf/robot_desherbor.urdf.xacro (robot description, xacro)
@@ -22,5 +22,5 @@
       <origin xyz="0 0 .1" rpy="0 0 0"/>
       <geometry>
-        <box size="0.1 0.3 0.1"/>
+        <box size="0.3 0.1 0.1"/>
       </geometry>
     </collision>

Commit message: modification detection herbe

File: desherbor_ensta/urdf/robot_desherbor.urdf.xacro (robot description, xacro)
@@ -20,5 +20,5 @@
   <link name="chassis">
     <collision>
-      <origin xyz="0 0 .1" rpy="0 0 0"/>
+      <origin xyz="0 0 0.1" rpy="0 0 0"/>
       <geometry>
         <box size="0.3 0.3 0.1"/>
@@ -26,5 +26,5 @@
     </collision>
     <visual>
-      <origin xyz="0 0 .1" rpy="0 0 0"/>
+      <origin xyz="0 0 0.1" rpy="0 0 0"/>
       <geometry>
         <box size="0.1 0.3 0.1"/>

Commit message: correction inertie roues arrieres et limites pour roues avants

File: desherbor_ensta/urdf/robot_desherbor.urdf.xacro (robot description, xacro)
@@ -6,8 +6,20 @@
   <xacro:include filename="$(find desherbor_ensta)/urdf/robot.lidar.xacro"/>
   <xacro:include filename="$(find desherbor_ensta)/urdf/robot.IMU.xacro"/>
+  <xacro:macro name="box_inertial" params="mass height width depth">
+    <inertial>
+      <mass value="${mass}" />
+      <inertia ixx="${0.08*mass*(height*height + depth*depth)}" ixy="0.0" ixz="0.0" iyy="${0.08*mass*(width*width + depth*depth)}" iyz="0.0" izz="${0.08*mass*(width*width + height*height)}" />
+    </inertial>
+  </xacro:macro>
+  <xacro:macro name="cylinder_inertial" params="length mass radius">
+    <inertial>
+      <mass value="${mass}"/>
+      <inertia ixx = "${0.08*(mass)*(3*radius*radius + length*length)}" ixy="0.0" ixz="0.0" iyy="${0.08*(mass)*(3*radius*radius + length*length)}" iyz="0.0" izz="${0.5*mass*radius*radius}" />
+    </inertial>
+  </xacro:macro>
   <xacro:macro name="default_inertial" params="mass">
     <inertial>
-      <mass value="${mass}" />
-      <inertia ixx="0.01" ixy="0.0" ixz="0.0" iyy="0.01" iyz="0.0" izz="0.01" />
+      <mass value="${mass}"/>
+      <inertia ixx="0.1" ixy="0.0" ixz="0.0" iyy="0.1" iyz="0.0" izz="0.1" />
     </inertial>
   </xacro:macro>
@@ -22,5 +34,5 @@
       <origin xyz="0 0 0.1" rpy="0 0 0"/>
       <geometry>
-        <box size="0.3 0.1 0.1"/>
+        <box size="0.3 0.1  0.1"/>
       </geometry>
     </collision>
@@ -28,8 +40,8 @@
       <origin xyz="0 0 0.1" rpy="0 0 0"/>
       <geometry>
-        <box size="0.3 0.3 0.1"/>
-      </geometry>
-    </visual>
-    <xacro:default_inertial mass="4.0"/>
+        <box size="0.3 0.2 0.1"/>
+      </geometry>
+    </visual>
+    <xacro:box_inertial mass="1.0" height="0.3" width="0.2" depth="0.1"/>
   </link>
   <link name="left_top_wheel">
@@ -46,5 +58,5 @@
       </geometry>
     </visual>
-    <xacro:default_inertial mass="0.3"/>
+    <xacro:cylinder_inertial mass="1" length="0.05" radius="0.1" />
   </link>
   <link name="right_top_wheel">
@@ -61,5 +73,5 @@
       </geometry>
     </visual>
-    <xacro:default_inertial mass="0.3"/>
+    <xacro:cylinder_inertial mass="1" length="0.05" radius="0.1" />
   </link>
   <link name="left_bottom_wheel">
@@ -76,5 +88,5 @@
       </geometry>
     </visual>
-    <xacro:default_inertial mass="0.3"/>
+    <xacro:cylinder_inertial mass="1" length="0.05" radius="0.1" />
   </link>
   <link name="right_bottom_wheel">
@@ -91,17 +103,19 @@
       </geometry>
     </visual>
-    <xacro:default_inertial mass="0.3"/>
-  </link>
-  <joint type="continuous" name="left_top_wheel_hinge">
+    <xacro:cylinder_inertial mass="1" length="0.05" radius="0.1" />
+  </link>
+  <joint type="revolute" name="left_top_wheel_hinge">
     <origin xyz="0.1 0.13 0.1" rpy="0 0 0"/>
     <child link="left_top_wheel"/>
     <parent link="chassis"/>
     <axis xyz="0 0 1"/>
-  </joint>
-  <joint type="continuous" name="right_top_wheel_hinge">
+    <limit effort="1000.0" lower="-0.78" upper="0.78" velocity="1.0" />
+  </joint>
+  <joint type="revolute" name="right_top_wheel_hinge">
     <origin xyz="0.1 -0.13 0.1" rpy="0 0 0"/>
     <child link="right_top_wheel"/>
     <parent link="chassis"/>
     <axis xyz="0 0 1"/>
+    <limit effort="1000.0" lower="-0.78" upper="0.78" velocity="1.0" />
   </joint>
   <joint type="continuous" name="left_bottom_wheel_hinge">
@@ -130,5 +144,5 @@
       </geometry>
     </visual>
-    <xacro:default_inertial mass="0.1"/>
+    <xacro:default_inertial mass=" 0.1"/>
   </link>
   <joint type="continuous" name="arm_hinge">

Commit message: Ajout des subscribers

File: desherbor_ensta/urdf/robot_desherbor.urdf.xacro (robot description, xacro)
@@ -210,5 +210,5 @@
   <link name="lidar">
     <visual>
-      <origin xyz="0 0 0.075" rpy="0 0 0"/>
+      <origin xyz="0 0 -0.03" rpy="0 0 0"/>
       <geometry>
         <cylinder radius="0.03" length="0.1"/>
@@ -219,6 +219,6 @@
   <joint name="lidar_hinge" type="fixed">
     <child link="lidar"/>
-    <parent link="arm"/>
-    <origin xyz="0 0 0.075" rpy="0 0 0"/>
+    <parent link="chassis"/>
+    <origin xyz="0 0 0.22" rpy="0 0 0"/>
   </joint>
     <link name="camera">
@@ -292,5 +292,5 @@
   <link name="imu_link">
     <visual>
-      <origin xyz="0 0 0.1" rpy="0 0 0"/>
+      <origin xyz="0 0 0.01" rpy="0 0 0"/>
       <geometry>
         <cylinder radius="0.01" length="0.01"/>

Commit message: tout fonctionne

File: desherbor_ensta/urdf/robot_desherbor.urdf.xacro (robot description, xacro)
@@ -107,15 +107,15 @@
   <joint type="revolute" name="left_top_wheel_hinge">
     <origin xyz="0.1 0.13 0.1" rpy="0 0 0"/>
-    <child link="left_top_wheel"/>
+    <child link="free_left"/>
     <parent link="chassis"/>
     <axis xyz="0 0 1"/>
-    <limit effort="1000.0" lower="-0.78" upper="0.78" velocity="1.0" />
+    <limit effort="1000.0" lower="-0.78" upper="0.78" velocity="10.0" />
   </joint>
   <joint type="revolute" name="right_top_wheel_hinge">
     <origin xyz="0.1 -0.13 0.1" rpy="0 0 0"/>
-    <child link="right_top_wheel"/>
+    <child link="free_right"/>
     <parent link="chassis"/>
     <axis xyz="0 0 1"/>
-    <limit effort="1000.0" lower="-0.78" upper="0.78" velocity="1.0" />
+    <limit effort="1000.0" lower="-0.78" upper="0.78" velocity="10.0" />
   </joint>
   <joint type="continuous" name="left_bottom_wheel_hinge">
@@ -131,4 +131,34 @@
     <axis xyz="0 1 0"/>
   </joint>
+  <joint type="continuous" name="free_right_top">
+    <origin xyz="0 0 0" rpy="0 0 0"/>
+    <child link="right_top_wheel"/>
+    <parent link="free_right"/>
+    <axis xyz="0 1 0"/>
+  </joint>
+  <joint type="continuous" name="free_left_top">
+    <origin xyz="0 0 0" rpy="0 0 0"/>
+    <child link="left_top_wheel"/>
+    <parent link="free_left"/>
+    <axis xyz="0 1 0"/>
+  </joint>
+  <link name="free_right">
+    <visual>
+      <origin xyz="0 0 0" rpy="0 0 0"/>
+      <geometry>
+        <cylinder radius="0.01" length="0.01"/>
+      </geometry>
+    </visual>
+    <xacro:default_inertial mass="0.1"/>
+  </link>
+  <link name="free_left">
+    <visual>
+      <origin xyz="0 0 0" rpy="0 0 0"/>
+      <geometry>
+        <cylinder radius="0.01" length="0.01"/>
+      </geometry>
+    </visual>
+    <xacro:default_inertial mass="0.1"/>
+  </link>
   <link name="arm">
     <collision>
@@ -211,5 +241,5 @@
     </joint>
     <actuator name="bottom_wheel_actuator">
-      <mechanicalReduction>50</mechanicalReduction>
+      <mechanicalReduction>10</mechanicalReduction>
       <hardwareInterface>EffortJointInterface</hardwareInterface>
     </actuator>
@@ -221,5 +251,5 @@
     </joint>
     <actuator name="bottom_wheel_actuator">
-      <mechanicalReduction>50</mechanicalReduction>
+      <mechanicalReduction>10</mechanicalReduction>
       <hardwareInterface>EffortJointInterface</hardwareInterface>
     </actuator>
@@ -230,5 +260,5 @@
       <hardwareInterface>EffortJointInterface</hardwareInterface>
     </joint>
-    <actuator name="top_wheel_actuator">
+    <actuator name="righttop_wheel_actuator">
       <mechanicalReduction>30</mechanicalReduction>
       <hardwareInterface>EffortJointInterface</hardwareInterface>
