Commit message: commande en position semi-fonctionelle

File: desherbor_ensta/urdf/robot.camera.xacro (robot description, xacro)
@@ -4,5 +4,5 @@
   <gazebo reference="camera">
     <sensor type="camera" name="main_camera">
-      <update_rate>3.0</update_rate>
+      <update_rate>20.0</update_rate>
       <camera name="head">
         <horizontal_fov>1.3962634</horizontal_fov>

File: desherbor_ensta/urdf/robot_desherbor.urdf.xacro (robot description, xacro)
@@ -43,5 +43,5 @@
       </geometry>
     </visual>
-    <xacro:box_inertial mass="10.0" height="0.3" width="0.2" depth="0.1"/>
+    <xacro:box_inertial mass="5.0" height="0.3" width="0.2" depth="0.1"/>
   </link>
   <link name="left_top_wheel">
@@ -58,5 +58,5 @@
       </geometry>
     </visual>
-    <xacro:cylinder_inertial mass="1" length="0.05" radius="0.1" />
+    <xacro:cylinder_inertial mass="0.1" length="0.05" radius="0.1" />
   </link>
   <link name="right_top_wheel">
@@ -73,5 +73,5 @@
       </geometry>
     </visual>
-    <xacro:cylinder_inertial mass="1" length="0.05" radius="0.1" />
+    <xacro:cylinder_inertial mass="0.1" length="0.05" radius="0.1" />
   </link>
   <link name="left_bottom_wheel">
@@ -88,5 +88,5 @@
       </geometry>
     </visual>
-    <xacro:cylinder_inertial mass="1" length="0.05" radius="0.1" />
+    <xacro:cylinder_inertial mass="0.1" length="0.05" radius="0.1" />
   </link>
   <link name="right_bottom_wheel">
@@ -103,5 +103,5 @@
       </geometry>
     </visual>
-    <xacro:cylinder_inertial mass="1" length="0.05" radius="0.1" />
+    <xacro:cylinder_inertial mass="0.1" length="0.05" radius="0.1" />
   </link>
   <joint type="revolute" name="left_top_wheel_hinge">
@@ -124,4 +124,5 @@
     <parent link="chassis"/>
     <axis xyz="0 1 0"/>
+    <dynamics damping ="0.3" friction="0.3"/>
   </joint>
   <joint type="continuous" name="right_bottom_wheel_hinge">
@@ -130,4 +131,5 @@
     <parent link="chassis"/>
     <axis xyz="0 1 0"/>
+    <dynamics damping ="0.3" friction="0.3"/>
   </joint>
   <joint type="continuous" name="free_right_top">
